File: alps64.kicad_pcb (KiCad board)
At the start: 2 copper layers, 285 x 95.2 mm, 200 parts, among them J1 USB_mini_micro_B, K00 KEYSW, K00_1 KEYSW, K00_2 KEYSW, K00_3 KEYSW, K01 KEYSW, K02 KEYSW, K03 KEYSW, K04 KEYSW, K05 KEYSW, K06 KEYSW, K07 KEYSW, K10 KEYSW, K10_1 KEYSW, K10_2 KEYSW, K11 KEYSW, K12 KEYSW, K13 KEYSW, K14 KEYSW, K15 KEYSW, K16 KEYSW, K17 KEYSW, K20 KEYSW, K20_1 KEYSW, K21 KEYSW, K21_1 KEYSW, K22 KEYSW, K23 KEYSW, K23_1 KEYSW, K23_2 KEYSW, K23_3 KEYSW, K24 KEYSW, K24_1 KEYSW, K25 KEYSW, K26 KEYSW, K27 KEYSW, K27_1 KEYSW, K30 KEYSW, K30_1 KEYSW, K31 KEYSW, K31_1 KEYSW, K32 KEYSW, K32_1 KEYSW, K32_2 ALPS_SKCM, K33 KEYSW, K34 KEYSW, K35 KEYSW, K36 KEYSW, K37 KEYSW, K40 KEYSW, K40_1 KEYSW, K40_2 KEYSW, K41 KEYSW, K42 KEYSW, K43 KEYSW, K44 KEYSW, K45 KEYSW, K46 KEYSW, K47 KEYSW, K50 KEYSW, K50_1 KEYSW, K50_2 KEYSW, K51 KEYSW, K52 KEYSW, K53 KEYSW, K54 KEYSW, K55 KEYSW, K56 KEYSW, K57 KEYSW, K60 KEYSW, K60_1 KEYSW, K60_2 KEYSW, K61 KEYSW, K62 KEYSW, K63 KEYSW, K64 KEYSW, K65 KEYSW, K66 KEYSW, K67 KEYSW, K70 KEYSW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

Commit message: first untested iteration for SpaceCadet mini
Parts:
- removed the D00 at (238.1, 90.5)
- removed the D10 at (259.6, 90.5)
- removed the D20 at (285.8, 90.5)
- removed K00, K00_3, K10_1, K20, K30, K40, K50: KEYSW, keyboard_parts:ALPS_SKCM_reverse_pad
- removed K00_2, K10_2, K40_1, K50_1: KEYSW, keyboard_parts:ALPS_SKCM
- removed the Poker_oval_hole at (265.1, 90.5)
- removed the Poker_oval_hole at (30.1, 90.5)
- moved D50 23.5 mm to (57.8, 86.5), turned to 180 degrees
- moved D00 18.0 mm to (241.8, 82.7), turned to 0 degrees
- moved D40 15.0 mm to (39.8, 90.5)
- moved K50_2 14.2 mm to (52.5, 90.5)
- moved K00_1 11.9 mm to (242.8, 90.5)
- moved D10 10.8 mm to (260.8, 82.6), turned to 0 degrees
- moved K10 9.51 mm to (261.9, 90.5)
- moved K40_2 9.46 mm to (33.4, 90.5)
- moved K20_1 2.37 mm to (281.0, 90.5)
- moved K30_1 2.34 mm to (14.3, 90.5)
Routing:
- net /matrix/col0: track 436.1 -> 345.4 mm
- net Net-(D00-Pad1): track 39.8 -> 11.9 mm
- net /matrix/row5: track 171.2 -> 193.7 mm
- net Net-(D10-Pad1): track 31.1 -> 12.0 mm
- net /matrix/row1: track 295.6 -> 277.3 mm
- net Net-(D50-Pad1): track 25.0 -> 8.50 mm
- net /matrix/row2: track 419.6 -> 405.8 mm
- net /matrix/row4: track 204.8 -> 218.5 mm
- net /matrix/row0: track 270.8 -> 257.5 mm
- net Net-(D40-Pad1): track 24.7 -> 12.4 mm
- net Net-(D20-Pad1): track 26.8 -> 14.8 mm
- net /matrix/row3: track 311.2 -> 318.8 mm
- net Net-(D30-Pad1): track 27.0 -> 32.1 mm
- net Net-(D34-Pad1): track 15.4 -> 14.2 mm
- net GND: track 337.9 -> 337.2 mm
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Other:
- net class 20mil removed
- net class 6mil removed
- net class 8mil removed
- net class Default removed
- net class Power removed

Commit message: Switch alignment correction
Parts:
- moved K50_2 0.10 mm to (52.4, 90.5)
- moved K40_2 0.06 mm to (33.3, 90.5)
Changed lines of the file:
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@@
       (usegerberattributes false)
       (usegerberadvancedattributes false)
-      (creategerberjobfile false)
+      (creategerberjobfile true)
       (svguseinch false)
       (svgprecision 6)
@@
   )
   (footprint "keyboard_parts:ALPS_SKCM" (layer "F.Cu")
-    (at 280.9748 90.4748 180)
+    (at 280.9875 90.4875 180)
     (descr "http://deskthority.net/wiki/File:Alps_Electric_--_spec_--_5454_31.pdf")
     (tags "ALPS, keyboard switch, SKCM, SKCL")
@@
   )
   (footprint "keyboard_parts:ALPS_SKCM_reverse_pad" (layer "F.Cu")
-    (at 261.9248 90.4748 180)
+    (at 261.9375 90.4875 180)
     (descr "http://deskthority.net/wiki/File:Alps_Electric_--_spec_--_5454_31.pdf")
     (tags "ALPS, keyboard switch, SKCM, SKCL")
@@
   )
   (footprint "keyboard_parts:ALPS_SKCM_reverse_pad" (layer "F.Cu")
-    (at 52.4764 90.5256 180)
+    (at 52.3875 90.4875 180)
     (descr "http://deskthority.net/wiki/File:Alps_Electric_--_spec_--_5454_31.pdf")
     (tags "ALPS, keyboard switch, SKCM, SKCL")
@@
   )
   (footprint "keyboard_parts:ALPS_SKCM_reverse_pad" (layer "F.Cu")
-    (at 242.8494 90.4875 180)
+    (at 242.8875 90.4875 180)
     (descr "http://deskthority.net/wiki/File:Alps_Electric_--_spec_--_5454_31.pdf")
     (tags "ALPS, keyboard switch, SKCM, SKCL")
@@
   )
   (footprint "keyboard_parts:ALPS_SKCM" (layer "F.Cu")
-    (at 14.3256 90.5002 180)
+    (at 14.2875 90.4875 180)
     (descr "http://deskthority.net/wiki/File:Alps_Electric_--_spec_--_5454_31.pdf")
     (tags "ALPS, keyboard switch, SKCM, SKCL")
@@
   )
   (footprint "keyboard_parts:ALPS_SKCM" (layer "F.Cu")
-    (at 33.401 90.4875 180)
-    (descr "http://deskthority.net/wiki/File:Alps_Electric_--_spec_--_5454_31.pdf")
-    (tags "ALPS, keyboard switch, SKCM, SKCL")
+    (at 33.3375 90.4875 180)
+    (descr "http://deskthority.net/wiki/File:Alps_Electric_--_spec_--_5454_31.pdf")
+    (tags "ALPS, keyboard switch, SKCM, SKCL")

Commit message: Rev A
First revision with revised bottom row created
Parts:
- removed G***: LOGO, keyboard_parts:tmk_logo
Other:
- board text added: "SpaceCadetSaver Rev.A darkcruix aka Roland Huber based on TMK Alps64 Rev.H"
- board text added: "created 2022-11"
- board text removed: "TMK Alps64 Rev.H"
- board text removed: "tmk-kbd.com"
